File: kicad/digital-control.sch (KiCad schematic (older format))
At the start: 30 parts, among them J3 CONN_01X04, Q3 MMBT3904, SW1 SPST, SW2 SPST, U4 STM32F031G, U5 SSD1306-OLED-I2C, U6 MMA8652FC

Commit message: Completed initial routing
Connections:
- net GND: now also SW2.2; no longer SW2.1
- net HEATER_LATCH_RESET: now also U4.12 (PA6); no longer U4.25 (PB4)
- net SW_B: now also SW2.1; no longer SW2.2
Changed lines of the file:
@@
 Text Label 5100 4700 0    60   ~ 0
 BUZ_COL
-Text HLabel 4300 3200 0    60   Input ~ 0
+Text HLabel 7500 2300 2    60   Input ~ 0
 HEATER_LATCH_RESET
 $Comp
@@
 	1    0    0    -1
 $EndComp
-Wire Wire Line
-	4900 2900 4400 2900
-Wire Wire Line
-	4400 2900 4400 3200
-Wire Wire Line
-	4400 3200 4300 3200
 NoConn ~ 6300 2600
 $Comp
@@
 F 4 "P15502CT-ND" H 1650 4600 60  0001 C CNN "Part No."
 	1    1650 4600
-	1    0    0    -1
+	-1   0    0    -1
 $EndComp
 Wire Wire Line
@@
 NoConn ~ 6300 2100
 NoConn ~ 6300 2200
-NoConn ~ 6300 2300
+Wire Wire Line
+	6300 2300 7500 2300
+NoConn ~ 4900 2900
 $EndSCHEMATC
